File: Kicad_Files/VESC-6-MK5/VESC-6-MK5.kicad_sch (KiCad schematic)
At the start: 37 parts, among them P1 USB_OTG, P2 CAN, P4 HALL_ENC, P5 COMM, P6 SERVO, P7 SWD, U11 SENSOR_VOLTAGE

Commit message: Working sample of the display
Parts:
- removed C32: 100u, DRV8301_:CAP_TPS1210_3P5X2P8_AVX, symbol Device:C_Polarized
Other:
- note removed: "Just using the footprint of this capacitor to connect PWR_GND and regular GND. I'll solder a wire across it on the final PCB"
Changed lines of the file:
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@@
-    (stroke (width 0) (type default))
-  )
-  (wire (pts (xy 39.37 168.91) (xy 46.99 168.91))
     (stroke (width 0) (type default))
   )
@@
     (stroke (width 0) (type default))
   )
-  (wire (pts (xy 46.99 168.91) (xy 46.99 171.45))
-    (stroke (width 0) (type default))
-  )
   (wire (pts (xy 101.6 149.86) (xy 104.14 149.86))
     (stroke (width 0) (type default))
@@
     (stroke (width 0) (type default))
   )
-  (wire (pts (xy 39.37 173.99) (xy 39.37 168.91))
-    (stroke (width 0) (type default))
-  )
   (wire (pts (xy 190.5 120.65) (xy 198.12 120.65))
     (stroke (width 0) (type default))
@@
   (wire (pts (xy 100.33 92.71) (xy 102.87 92.71))
     (stroke (width 0) (type default))
-  )
-  (text "Just using the footprint of this capacitor\nto connect PWR_GND and regular GND.\nI'll solder a wire across it on the final PCB"
-    (at 17.78 166.37 0)
-    (effects (font (size 1.27 1.27)) (justify left bottom))
   )
   (text "Optional" (at 105.41 24.13 0)
@@
     )
   )
-  (symbol (lib_id "power:GND") (at 46.99 179.07 0) (unit 1)
-    (in_bom yes) (on_board yes) (dnp no) (fields_autoplaced)
-    (property "Reference" "#PWR097" (at 46.99 185.42 0)
-      (effects (font (size 1.27 1.27)) hide)
-    )
-    (property "Value" "GND" (at 46.99 184.15 0)
-      (effects (font (size 1.27 1.27)))
-    )
-    (property "Footprint" "" (at 46.99 179.07 0)
-      (effects (font (size 1.27 1.27)) hide)
-    )
-    (property "Datasheet" "" (at 46.99 179.07 0)
-      (effects (font (size 1.27 1.27)) hide)
-    )
-    (pin "1")
-    (instances
-      (project "VESC-6-MK5"
-        (path "/2841ac42-8ec3-4366-9083-5e27f86f2676"
-          (reference "#PWR097") (unit 1)
-        )
-      )
-    )
-  )
   (symbol (lib_id "Device:R") (at 111.76 29.21 90) (unit 1)
     (in_bom yes) (on_board yes) (dnp no)
@@
         (path "/2841ac42-8ec3-4366-9083-5e27f86f2676"
           (reference "#PWR088") (unit 1)
-        )
-      )
-    )
-  )
-  (symbol (lib_id "Device:C_Polarized") (at 46.99 175.26 0) (unit 1)
-    (in_bom yes) (on_board yes) (dnp no) (fields_autoplaced)
-    (property "Reference" "C32" (at 50.8 173.736 0)
-      (effects (font (size 1.27 1.27)) (justify left))
-    )
-    (property "Value" "100u" (at 50.8 176.276 0)
-      (effects (font (size 1.27 1.27)) (justify left))
-    )
-    (property "Footprint" "DRV8301_:CAP_TPS1210_3P5X2P8_AVX" (at 47.9552 179.07 0)
-      (effects (font (size 1.27 1.27)) hide)
-    )
-    (property "Datasheet" "~" (at 46.99 175.26 0)
-      (effects (font (size 1.27 1.27)) hide)
-    )
-    (pin "1")
-    (pin "2")
-    (instances
-      (project "VESC-6-MK5"
-        (path "/2841ac42-8ec3-4366-9083-5e27f86f2676/7f79de6f-9a46-4274-b1b5-000aa0200c27"
-          (reference "C32") (unit 1)
-        )
-        (path "/2841ac42-8ec3-4366-9083-5e27f86f2676"
-          (reference "C60") (unit 1)
         )
       )
@@
         )
       )
-    )
-  )
-  (symbol (lib_id "power:GNDPWR") (at 39.37 173.99 0) (unit 1)
-    (in_bom yes) (on_board yes) (dnp no) (fields_autoplaced)
-    (property "Reference" "#PWR025" (at 39.37 179.07 0)
-      (effects (font (size 1.27 1.27)) hide)
-    )
-    (property "Value" "GNDPWR" (at 39.243 177.8 0)
-      (effects (font (size 1.27 1.27)))
-    )
-    (property "Footprint" "" (at 39.37 175.26 0)
-      (effects (font (size 1.27 1.27)) hide)
-    )
-    (property "Datasheet" "" (at 39.37 175.26 0)
-      (effects (font (size 1.27 1.27)) hide)
-    )
-    (pin "1")
-    (instances
-      (project "VESC-6-MK5"
-        (path "/2841ac42-8ec3-4366-9083-5e27f86f2676/9bfd20ee-39f5-4017-8cd2-0d9172ead4cb"
-          (reference "#PWR025") (unit 1)
-        )
-        (path "/2841ac42-8ec3-4366-9083-5e27f86f2676"
-          (reference "#PWR098") (unit 1)
-        )
-      )
