File: Receiver/Receiver_KiCad/MCU.kicad_sch (KiCad schematic)
At the start: 21 parts, among them J3 61300511121, J4 M20-9990246, U3 STM32G030F6Px, U4 NRF24L01_Breakout

Commit message: Finished Receiver V1
Parts:
- removed J4: M20-9990246, MCU_:CONN2_M20-999_1x2_HRW, symbol M20-9990246:M20-9990246
- removed R5: 4.7k, Power_:RESC1005X40N, symbol Device:R
- removed S2: TL1105BF160Q, MCU_:SW_TL1105BF160Q, symbol TL1105BF160Q:TL1105BF160Q
- removed U10, U11, U12, U13, U14, U15, U5, U6, U7, U8, U9: ~, MCU_:Wire_Via, symbol Via:Small_Via
- removed U3: STM32G030F6Px, Package_SO:TSSOP-20_4.4x6.5mm_P0.65mm, symbol MCU_ST_STM32G0:STM32G030F6Px
- added J1: B3B-XH-A, MCU_:JST_B3B-XH-A, symbol B3B-XH-A:B3B-XH-A
- added J2: 61300311121, MCU_:WURTH_61300311121, symbol 61300311121:61300311121
- added J3: B5B-PH-K-S, MCU_:JST_B5B-PH-K-S, symbol B5B-PH-K-S:B5B-PH-K-S
- added R1, R2: 4.7k, MCU_:RESC1508X55N, symbol Device:R
- added U1: STM32G031F8Px, Package_SO:TSSOP-20_4.4x6.5mm_P0.65mm, symbol MCU_ST_STM32G0:STM32G031F8Px
- added U2: FM24CL16B, Package_SO:SOIC-8_3.9x4.9mm_P1.27mm, symbol Memory_NVRAM:FM24CL16B
- renumbered C5 to C1, C6 to C2, D3 to D1, J3 to J4, R4 to R3, U4 to U3
Connections:
- net GND: now also J1.1, J2.01, J3.3, U1.5 (VSS), U2.4 (VSS)
- net SPI1_CE: now also U1.10 (PA3)
- net SPI1_CSN: now also U1.11 (PA4)
- net SPI1_MISO: now also U1.13 (PA6)
- net SPI1_MOSI: now also U1.9 (PA2)
- net SPI1_SCK: now also U1.8 (PA1)
- net VDD: now also J3.2, R1.1, R2.1, U1.4 (VDD), U2.8 (VDD)
- net at J4.2: now also U1.18 (PA13)
- net at J4.3: now also U1.19 (PA14/PA15)
- net at J4.4: now also U1.6 (PF2)
- net SPI1_IRQ: now reaches U3.8 (IRQ)
- net SPI1_IRQ: now also U1.12 (PA5)
- net GPIO_Output renamed STATUS_LED
- net STATUS_LED: now also U1.14 (PA7)
- new net +5V: J1.2, J2.03, J3.1
- new net I2C_SCL: R1.2, U1.16 (PA11/PA9), U2.6 (SCL)
- new net I2C_SDA: R2.2, U1.17 (PA12/PA10), U2.5 (SDA)
- new net PWM_OUT: J1.3, U1.15 (PB0/PB1/PB2/PA8)
- new net SK6812_OUT: J2.02, U1.3 (PC15)
- new net UART1_RX: J3.4, U1.1 (PB7/PB8)
- new net UART1_TX: J3.5, U1.20 (PB3/PB4/PB5/PB6)
- new net WP: U1.2 (PC14/PB9), U2.7 (WP)
- no-connect marks 1 -> 0
Other:
- note added: "External Memory"
- note added: "LED Strip"
- note added: "NRST"
- note added: "PWM Output"
- note added: "SWD"
- note added: "UART Port/5v In"
- note added: "Wireless Module"
- note removed: "Vias For LCD Module"
- note removed: "Vias for joystick"
- moved on the sheet: D1, J4, R3
