File: Receiver/Receiver_KiCad/Power.kicad_sch (KiCad schematic)
At the start: 3 parts, among them J2 B2B-XH-A

Commit message: Finished Receiver V1
Parts:
- removed J2: B2B-XH-A, Power_:JST_B2B-XH-A, symbol B2B-XH-A:B2B-XH-A
- removed R1: 100k, symbol Device:R
- removed R2: 7k, symbol Device:R
Changed lines of the file:
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@@
 (kicad_sch (version 20230121) (generator eeschema)
   (paper "A4")
-  (junction (at 113.03 71.12) (diameter 0) (color 0 0 0 0)
-  )
-  (junction (at 124.46 71.12) (diameter 0) (color 0 0 0 0)
-  )
-  (wire (pts (xy 107.95 71.12) (xy 113.03 71.12))
-    (stroke (width 0) (type default))
-  )
-  (wire (pts (xy 113.03 66.04) (xy 113.03 71.12))
-    (stroke (width 0) (type default))
-  )
-  (wire (pts (xy 124.46 71.12) (xy 128.27 71.12))
-    (stroke (width 0) (type default))
-  )
-  (wire (pts (xy 113.03 71.12) (xy 116.84 71.12))
-    (stroke (width 0) (type default))
-  )
-  (wire (pts (xy 107.95 69.85) (xy 107.95 71.12))
-    (stroke (width 0) (type default))
-  )
-  (wire (pts (xy 138.43 71.12) (xy 138.43 73.66))
-    (stroke (width 0) (type default))
-  )
-  (wire (pts (xy 135.89 71.12) (xy 138.43 71.12))
-    (stroke (width 0) (type default))
-  )
-  (wire (pts (xy 124.46 71.12) (xy 124.46 74.93))
-    (stroke (width 0) (type default))
-  )
-  (hierarchical_label "ADC" (shape output) (at 124.46 74.93 270) (fields_autoplaced)
-    (effects (font (size 1.27 1.27)) (justify right))
-  )
-  (symbol (lib_id "power:GND") (at 115.57 66.04 0) (unit 1)
-    (in_bom yes) (on_board yes) (dnp no)
-    (property "Reference" "#PWR02" (at 115.57 72.39 0)
-      (effects (font (size 1.27 1.27)) hide)
-    )
-    (property "Value" "GND" (at 118.11 66.04 0)
-      (effects (font (size 1.27 1.27)))
-    )
-    (property "Footprint" "" (at 115.57 66.04 0)
-      (effects (font (size 1.27 1.27)) hide)
-    )
-    (property "Datasheet" "" (at 115.57 66.04 0)
-      (effects (font (size 1.27 1.27)) hide)
-    )
-    (pin "1")
-    (instances
-      (project "Receiver_KiCad"
-        (path "/b4382ef4-8540-4cf0-8bf7-60a21f991ddf/d6ef35f0-db14-4fb6-a886-f39262892cda"
-          (reference "#PWR02") (unit 1)
-        )
-      )
-    )
-  )
-  (symbol (lib_id "power:GND") (at 138.43 73.66 0) (unit 1)
-    (in_bom yes) (on_board yes) (dnp no)
-    (property "Reference" "#PWR01" (at 138.43 80.01 0)
-      (effects (font (size 1.27 1.27)) hide)
-    )
-    (property "Value" "GND" (at 140.97 73.66 0)
-      (effects (font (size 1.27 1.27)))
-    )
-    (property "Footprint" "" (at 138.43 73.66 0)
-      (effects (font (size 1.27 1.27)) hide)
-    )
-    (property "Datasheet" "" (at 138.43 73.66 0)
-      (effects (font (size 1.27 1.27)) hide)
-    )
-    (pin "1")
-    (instances
-      (project "Receiver_KiCad"
-        (path "/b4382ef4-8540-4cf0-8bf7-60a21f991ddf/d6ef35f0-db14-4fb6-a886-f39262892cda"
-          (reference "#PWR01") (unit 1)
-        )
-      )
-    )
-  )
-  (symbol (lib_id "Device:R") (at 120.65 71.12 90) (unit 1)
-    (in_bom yes) (on_board yes) (dnp no)
-    (property "Reference" "R1" (at 120.65 68.58 90)
-      (effects (font (size 1.27 1.27)))
-    )
-    (property "Value" "100k" (at 120.65 71.12 90)
-      (effects (font (size 1.27 1.27)))
-    )
-    (property "Footprint" "" (at 120.65 72.898 90)
-      (effects (font (size 1.27 1.27)) hide)
-    )
-    (property "Datasheet" "~" (at 120.65 71.12 0)
-      (effects (font (size 1.27 1.27)) hide)
-    )
-    (pin "1")
-    (pin "2")
-    (instances
-      (project "Receiver_KiCad"
-        (path "/b4382ef4-8540-4cf0-8bf7-60a21f991ddf/d6ef35f0-db14-4fb6-a886-f39262892cda"
-          (reference "R1") (unit 1)
-        )
-      )
-    )
-  )
-  (symbol (lib_id "B2B-XH-A:B2B-XH-A") (at 115.57 58.42 90) (unit 1)
-    (in_bom yes) (on_board yes) (dnp no) (fields_autoplaced)
-    (property "Reference" "J2" (at 119.38 57.15 90)
-      (effects (font (size 1.27 1.27)) (justify right))
-    )
-    (property "Value" "B2B-XH-A" (at 119.38 59.69 90)
-      (effects (font (size 1.27 1.27)) (justify right))
-    )
-    (property "Footprint" "Power_:JST_B2B-XH-A" (at 115.57 58.42 0)
-      (effects (font (size 1.27 1.27)) (justify bottom) hide)
-    )
-    (property "Datasheet" "" (at 115.57 58.42 0)
-      (effects (font (size 1.27 1.27)) hide)
-    )
-    (property "PARTREV" "N/A" (at 115.57 58.42 0)
-      (effects (font (size 1.27 1.27)) (justify bottom) hide)
-    )
-    (property "STANDARD" "Manufacturer Recommendations" (at 115.57 58.42 0)
-      (effects (font (size 1.27 1.27)) (justify bottom) hide)
-    )
-    (property "MAXIMUM_PACKAGE_HEIGHT" "7 mm" (at 115.57 58.42 0)
-      (effects (font (size 1.27 1.27)) (justify bottom) hide)
-    )
-    (property "MANUFACTURER" "JST Sales America Inc." (at 115.57 58.42 0)
-      (effects (font (size 1.27 1.27)) (justify bottom) hide)
-    )
-    (pin "1")
-    (pin "2")
-    (instances
-      (project "Receiver_KiCad"
-        (path "/b4382ef4-8540-4cf0-8bf7-60a21f991ddf/d6ef35f0-db14-4fb6-a886-f39262892cda"
-          (reference "J2") (unit 1)
-        )
-      )
-    )
-  )
-  (symbol (lib_id "Device:R") (at 132.08 71.12 90) (unit 1)
-    (in_bom yes) (on_board yes) (dnp no)
-    (property "Reference" "R2" (at 132.08 68.58 90)
-      (effects (font (size 1.27 1.27)))
-    )
-    (property "Value" "7k" (at 132.08 71.12 90)
-      (effects (font (size 1.27 1.27)))
-    )
-    (property "Footprint" "" (at 132.08 72.898 90)
-      (effects (font (size 1.27 1.27)) hide)
-    )
-    (property "Datasheet" "~" (at 132.08 71.12 0)
-      (effects (font (size 1.27 1.27)) hide)
-    )
-    (pin "1")
-    (pin "2")
-    (instances
-      (project "Receiver_KiCad"
-        (path "/b4382ef4-8540-4cf0-8bf7-60a21f991ddf/d6ef35f0-db14-4fb6-a886-f39262892cda"
-          (reference "R2") (unit 1)
-        )
-      )
-    )
-  )
-  (symbol (lib_id "power:+BATT") (at 107.95 69.85 0) (unit 1)
-    (in_bom yes) (on_board yes) (dnp no) (fields_autoplaced)
-    (property "Reference" "#PWR03" (at 107.95 73.66 0)
-      (effects (font (size 1.27 1.27)) hide)
-    )
-    (property "Value" "+BATT" (at 107.95 64.77 0)
-      (effects (font (size 1.27 1.27)))
-    )
-    (property "Footprint" "" (at 107.95 69.85 0)
-      (effects (font (size 1.27 1.27)) hide)
-    )
-    (property "Datasheet" "" (at 107.95 69.85 0)
-      (effects (font (size 1.27 1.27)) hide)
-    )
-    (pin "1")
-    (instances
-      (project "Receiver_KiCad"
-        (path "/b4382ef4-8540-4cf0-8bf7-60a21f991ddf/d6ef35f0-db14-4fb6-a886-f39262892cda"
-          (reference "#PWR03") (unit 1)
-        )
-      )
-    )
-  )
 )
