File: Receiver/Receiver_KiCad/Receiver_KiCad.kicad_pcb (KiCad board)
At the start: 2 copper layers, 70.2 x 46.7 mm, 40 parts, among them J1 USB4125-GF-A_REVA2, J2 B2B-XH-A, J3 61300511121, J4 M20-9990246, U1 MCP73831T-2DCI_OT, U10 DIN, U11 CLK, U12 CS, U13 DC, U14 RST, U15 BL, U2 AP2210N-3.3TRG1, U3 STM32G030F6Px, U4 NRF24L01_Breakout, U5 ADC, U6 VDD, U7 GND, U8 VCC, U9 GND

Commit message: Finished Receiver V1
Parts:
- removed ? (x3): , 
- removed C3, C4, C5: 4u7, Power_:CAPC1608X90N
- removed C6: 100n, MCU_:CAPC1005X55N
- removed D3: LTST-C190GKT, MCU_:LEDC1608X35N
- removed D4: Charging, MCU_:0603
- removed R4: 120, MCU_:RESC2012X65N
- removed R5: 4.7k, Power_:RESC1005X40N
- removed R6, R7: 5.1k, Power_:RESC1608X50N
- removed S1: EG1218, Power_:SW_EG1218
- removed S2: TL1105BF160Q, MCU_:SW_TL1105BF160Q
- removed U10: DIN, MCU_:Wire_Via
- removed U11: CLK, MCU_:Wire_Via
- removed U12: CS, MCU_:Wire_Via
- removed U13: DC, MCU_:Wire_Via
- removed U14: RST, MCU_:Wire_Via
- removed U15: BL, MCU_:Wire_Via
- removed U4: NRF24L01_Breakout, RF_Module:nRF24L01_Breakout
- removed U5: ADC, MCU_:Wire_Via
- removed U6: VDD, MCU_:Wire_Via
- removed U7, U9: GND, MCU_:Wire_Via
- removed U8: VCC, MCU_:Wire_Via
- added G***: LOGO, MCU_:Skate3, F.Cu at (147.8, 142.1)
- added G***: LOGO, LOGO, B.Cu at (165.1, 139.5)
- C2: value 4u7 -> 100n; footprint Power_:CAPC1608X90N -> MCU_:CAPC1005X55N
- D1: value Ready -> LTST-C190GKT
- J1: value USB4125-GF-A_REVA2 -> B3B-XH-A; footprint Power_:GCT_USB4125-GF-A_REVA2 -> MCU_:JST_B3B-XH-A
- J2: value B2B-XH-A -> 61300311121; footprint Power_:JST_B2B-XH-A -> MCU_:WURTH_61300311121
- J3: value 61300511121 -> B5B-PH-K-S; footprint MCU_:CONN5_0511121_WRE -> MCU_:JST_B5B-PH-K-S
- J4: value M20-9990246 -> 61300511121; footprint MCU_:CONN2_M20-999_1x2_HRW -> MCU_:CONN5_0511121_WRE
- R1: value 5k -> 4.7k; footprint Power_:RESC3116X65N -> MCU_:RESC1508X55N
- R2: value 250 -> 4.7k; footprint Power_:RESC1608X55N -> MCU_:RESC1508X55N
- R3: value 250 -> 120; footprint Power_:RESC1608X55N -> MCU_:RESC2012X65N
- U1: value MCP73831T-2DCI_OT -> STM32G031F8Px; footprint Power_:SOT95P270X145-5N -> Package_SO:TSSOP-20_4.4x6.5mm_P0.65mm
- U2: value AP2210N-3.3TRG1 -> FM24CL16B; footprint Power_:SOT95P280X145-3N -> Package_SO:SOIC-8_3.9x4.9mm_P1.27mm
- U3: value STM32G030F6Px -> NRF24L01_Breakout; footprint Package_SO:TSSOP-20_4.4x6.5mm_P0.65mm -> RF_Module:nRF24L01_Breakout
- moved D1 67.2 mm to (165.5, 145.1), turned to 0 degrees
- moved R3 65.6 mm to (165.4, 140.2), turned to 0 degrees
- moved J1 65.6 mm to (176.5, 143.4), turned to 0 degrees
- moved J4 64.4 mm to (170.0, 119.6), turned to 0 degrees
- moved U2 53.0 mm to (177.0, 128.2), turned to 180 degrees
- moved U3 51.5 mm to (153.3, 125.1), turned to 0 degrees
- moved R2 50.3 mm to (169.9, 124.7), turned to -90 degrees
- moved C1 44.1 mm to (159.8, 127.7), turned to -90 degrees
- moved U1 39.7 mm to (164.7, 128.2), turned to 0 degrees
- moved R1 39.1 mm to (172.2, 124.7), turned to -90 degrees
- moved J2 36.9 mm to (148.0, 128.4)
- moved C2 34.3 mm to (158.2, 127.6), turned to 90 degrees
- moved J3 30.6 mm to (156.3, 118.0)
Connections:
- C1 pad 1: +5V -> VDD
- C2 pad 1: GND -> VDD
- C2 pad 2: +BATT -> GND
- J3 pad 1: VDD -> +5V
- J3 pad 2: Net-(U3-PA13) -> VDD
- J3 pad 3: Net-(U3-PA14/PA15) -> GND
- J3 pad 4: Net-(U3-NRST) -> /MCU/UART1_RX
- J3 pad 5: GND -> /MCU/UART1_TX
- J4 pad 1: GND -> VDD
- J4 pad 2: /MCU/USART1_TX -> Net-(U1-PA13)
- R1 pad 1: GND -> VDD
- R1 pad 2: Net-(U1-PROG) -> /MCU/I2C_SCL
- R2 pad 1: Net-(D4-Pad1) -> VDD
- R2 pad 2: Net-(U1-STAT) -> /MCU/I2C_SDA
- R3 pad 1: Net-(D1-PadA) -> /MCU/STATUS_LED
- R3 pad 2: Net-(U1-STAT) -> Net-(D1-PadA)
- U1 pad 1: Net-(U1-STAT) -> /MCU/UART1_RX
- U1 pad 2: GND -> /MCU/WP
- U1 pad 3: +BATT -> /MCU/SK6812_OUT
- U1 pad 4: +5V -> VDD
- U1 pad 5: Net-(U1-PROG) -> GND
- U2 pad 1: GND -> unconnected-(U2-Pad1)
- U2 pad 2: VDD -> unconnected-(U2-Pad2)
- U2 pad 3: Net-(U2-VIN) -> unconnected-(U2-Pad3)
- U3 pad 1: /MCU/Display_BL -> GND
- U3 pad 2: /MCU/SPI2_CS -> VDD
- U3 pad 3: /MCU/Display_DC -> /MCU/SPI1_CE
- U3 pad 4: VDD -> /MCU/SPI1_CSN
- U3 pad 5: GND -> /MCU/SPI1_SCK
- U3 pad 6: Net-(U3-NRST) -> /MCU/SPI1_MOSI
- U3 pad 7: /MCU/SPI2_SCK -> /MCU/SPI1_MISO
- U3 pad 8: /MCU/ADC1_IN1 -> /MCU/SPI1_IRQ
Routing:
- net +BATT: track 44.7 -> 0.00 mm
- net +5V: track 31.6 -> 73.3 mm
- net /MCU/SPI2_MOSI: track 38.9 -> 0.00 mm, vias 2 -> 0
- net /MCU/Display_RST: track 36.4 -> 0.00 mm
- net /MCU/ADC1_IN1: track 35.0 -> 0.00 mm, vias 1 -> 0
- net /MCU/SPI2_SCK: track 32.8 -> 0.00 mm
- net Net-(U3-PA14/PA15): track 32.6 -> 0.00 mm
- net Net-(U3-PA13): track 31.3 -> 0.00 mm, vias 2 -> 0
- net /MCU/SPI2_CS: track 30.8 -> 0.00 mm
- net /MCU/Display_DC: track 29.9 -> 0.00 mm
- net /MCU/Display_BL: track 28.6 -> 0.00 mm
- net Net-(U2-VIN): track 24.5 -> 0.00 mm
- net GND: track 28.9 -> 4.41 mm, vias 6 -> 0
- net Net-(U1-STAT): track 22.8 -> 0.00 mm
- net Net-(U1-PF2): track 0.00 -> 21.5 mm, vias 0 -> 2
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Other:
- board size 70.2 x 46.7 mm -> 38.5 x 35.7 mm
- board text added: "3V3"
- board text added: "5V"
- board text added: "CLK"
- board text added: "DIO"
- board text added: "LED"
- board text added: "PWM"
- board text added: "RX"
- board text added: "Receiver V1"
- board text removed: "+"
- board text removed: "-"
- board text removed: "1578 500mAh"
- board text removed: "3.3V"
- board text removed: "OFF"
- board text removed: "ON"
- board text removed: "Remote V1"
- board text removed: "SWCLK"
- board text removed: "SWDIO"
