File: Receiver/Receiver_KiCad/Receiver_KiCad.kicad_sch (KiCad schematic)
At the start: 0 parts

Commit message: Finished Receiver V1
Other:
- removed sheet Power
Changed lines of the file:
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@@
-    )
-  )
-  (sheet (at 86.36 63.5) (size 21.59 39.37) (fields_autoplaced)
-    (stroke (width 0.1524) (type solid))
-    (fill (color 0 0 0 0.0000))
-    (property "Sheetname" "Power" (at 86.36 62.7884 0)
-      (effects (font (size 1.27 1.27)) (justify left bottom))
-    )
-    (property "Sheetfile" "Power.kicad_sch" (at 86.36 103.4546 0)
-      (effects (font (size 1.27 1.27)) (justify left top))
-    )
-    (instances
-      (project "Receiver_KiCad"
-        (path "/b4382ef4-8540-4cf0-8bf7-60a21f991ddf" (page "2"))
-      )
     )
   )
